File: PCB/agricoltura-vine-k/Relay_Control.sch (KiCad schematic (older format))
At the start: 17 parts

Commit message: Relay and Board
Relay circuits added and exported to PCB
Parts:
- added C? (x2): C0402C104K9PACTU, AVR-KiCAD-Lib-Resistors:R0402, symbol AVR-KiCAD-Lib-Capacitors:C0402C104K9PACTU
- added D? (x2): LTST-C194TBKT, AVR-KiCAD-Lib-Diodes:LED0603, symbol AVR-KiCAD-Lib-Diodes:LTST-C194TBKT
- added D? (x2): B240A-13-F, AVR-KiCAD-Lib-Diodes:B240A-13-F, symbol AVR-KiCAD-Lib-Diodes:B240A-13-F
- added K? (x2): G5LE-14_DC5, AVR-KiCAD-Lib-Relays-Contactors:G5LE-14_DC5, symbol AVR-KiCAD-Lib-Mech-Relays-Contactors:G5LE-14_DC5
- added Q? (x2): IRLML6346TRPBF, AVR-KiCAD-Lib-Transistors:SOT-23, symbol AVR-KiCAD-Lib-Transistors:IRLML6346TRPBF
- added R? (x4): RC0402FR-0710RL, AVR-KiCAD-Lib-Resistors:R0402, symbol AVR-KiCAD-Lib-Diodes:RC0402FR-0710RL
- added T?: 0395121006, AVR-KiCAD-Lib-Connectors:0395121006, symbol AVR-KiCAD-Lib-Connectors:0395121006
- added U? (x2): ZXGD3009E6TA, growbox-KiCAD-ICs:SOT-23-6_Handsoldering, symbol AVR-KiCAD-Lib-ICs:ZXGD3009E6TA
Connections:
- net labels added: DRV3, DRV4
- wire segments 43 -> 86
Other:
- moved on the sheet: C?, D?, K?, Q?, R?, U?

Commit message: PCB Routing PRogress
5th relay added to schematic, PCB section with Relays routed, still need to connecto IO expander channels.
Parts:
- removed T? (x2): 0395121006, AVR-KiCAD-Lib-Connectors:0395121006, symbol AVR-KiCAD-Lib-Connectors:0395121006
- added C?: C0402C104K9PACTU, AVR-KiCAD-Lib-Resistors:R0402, symbol AVR-KiCAD-Lib-Capacitors:C0402C104K9PACTU
- added D12: B240A-13-F, AVR-KiCAD-Lib-Diodes:B240A-13-F, symbol AVR-KiCAD-Lib-Diodes:B240A-13-F
- added D13: LTST-C194TBKT, AVR-KiCAD-Lib-Diodes:LED0603, symbol AVR-KiCAD-Lib-Diodes:LTST-C194TBKT
- added K5: G5LE-14_DC5, AVR-KiCAD-Lib-Relays-Contactors:G5LE-14_DC5, symbol AVR-KiCAD-Lib-Mech-Relays-Contactors:G5LE-14_DC5
- added Q5: IRLML6346TRPBF, AVR-KiCAD-Lib-Transistors:SOT-23, symbol AVR-KiCAD-Lib-Transistors:IRLML6346TRPBF
- added R26, R27: RC0402FR-0710RL, AVR-KiCAD-Lib-Resistors:R0402, symbol AVR-KiCAD-Lib-Diodes:RC0402FR-0710RL
- added T4, T5, T6, T7, T8: 0395121003, AVR-KiCAD-Lib-Connectors:0395121003, symbol AVR-KiCAD-Lib-Connectors:0395121003
- added U11: ZXGD3009E6TA, growbox-KiCAD-ICs:SOT-23-6_Handsoldering, symbol AVR-KiCAD-Lib-ICs:ZXGD3009E6TA
- gave numbers to parts that had none: 32
Connections:
- wire segments 86 -> 99

Commit message: Finished
PCB routing complete, up for review before fab.
Parts:
- gave numbers to parts that had none: 1
Connections:
- net labels added: DRV5
Other:
- moved on the sheet: C36, D12, D13, K5, Q5, R26, R27, T8, U11

Commit message: PCB Tweaks
PCB tweaked for packaging in water resistant housing for greenhouse deployment
Parts:
- R18, R19, R20, R21, R22, R23, R24, R25, R26, R27: symbol AVR-KiCAD-Lib-Diodes:RC0402FR-0710RL -> agricoltura-vine-k-rescue:RC0402FR-0710RL-AVR-KiCAD-Lib-Diodes
Changed lines of the file:
@@
 $EndComp
 $Comp
-L AVR-KiCAD-Lib-Diodes:RC0402FR-0710RL R?
+L agricoltura-vine-k-rescue:RC0402FR-0710RL-AVR-KiCAD-Lib-Diodes R?
 U 1 1 5F02588D
 P 4100 1800
 AR Path="/5EF943A9/5F02588D" Ref="R?"  Part="1"
 AR Path="/5F0125AE/5F02588D" Ref="R19"  Part="1"
+AR Path="/5F02588D" Ref="R19"  Part="1"
 F 0 "R19" H 4100 1900 50  0000 C CNN
 F 1 "RC0402FR-0710RL" H 4100 2025 50  0001 C CNN
@@
 Connection ~ 3900 1800
 $Comp
-L AVR-KiCAD-Lib-Diodes:RC0402FR-0710RL R?
+L agricoltura-vine-k-rescue:RC0402FR-0710RL-AVR-KiCAD-Lib-Diodes R?
 U 1 1 5F0258AE
 P 4100 1500
 AR Path="/5EF943A9/5F0258AE" Ref="R?"  Part="1"
 AR Path="/5F0125AE/5F0258AE" Ref="R18"  Part="1"
+AR Path="/5F0258AE" Ref="R18"  Part="1"
 F 0 "R18" H 4100 1600 50  0000 C CNN
 F 1 "RC0402FR-0710RL" H 4100 1725 50  0001 C CNN
@@
 $EndComp
 $Comp
-L AVR-KiCAD-Lib-Diodes:RC0402FR-0710RL R?
+L agricoltura-vine-k-rescue:RC0402FR-0710RL-AVR-KiCAD-Lib-Diodes R?
 U 1 1 5F0258EC
 P 4100 3100
 AR Path="/5EF943A9/5F0258EC" Ref="R?"  Part="1"
 AR Path="/5F0125AE/5F0258EC" Ref="R21"  Part="1"
+AR Path="/5F0258EC" Ref="R21"  Part="1"
 F 0 "R21" H 4100 3200 50  0000 C CNN
 F 1 "RC0402FR-0710RL" H 4100 3325 50  0001 C CNN
@@
 Connection ~ 3900 3100
 $Comp
-L AVR-KiCAD-Lib-Diodes:RC0402FR-0710RL R?
+L agricoltura-vine-k-rescue:RC0402FR-0710RL-AVR-KiCAD-Lib-Diodes R?
 U 1 1 5F02590D
 P 4100 2800
 AR Path="/5EF943A9/5F02590D" Ref="R?"  Part="1"
 AR Path="/5F0125AE/5F02590D" Ref="R20"  Part="1"
+AR Path="/5F02590D" Ref="R20"  Part="1"
 F 0 "R20" H 4100 2900 50  0000 C CNN
 F 1 "RC0402FR-0710RL" H 4100 3025 50  0001 C CNN
@@
 $EndComp
 $Comp
-L AVR-KiCAD-Lib-Diodes:RC0402FR-0710RL R?
+L agricoltura-vine-k-rescue:RC0402FR-0710RL-AVR-KiCAD-Lib-Diodes R?
 U 1 1 5F02DC36
 P 4100 4650
 AR Path="/5EF943A9/5F02DC36" Ref="R?"  Part="1"
 AR Path="/5F0125AE/5F02DC36" Ref="R23"  Part="1"
+AR Path="/5F02DC36" Ref="R23"  Part="1"
 F 0 "R23" H 4100 4750 50  0000 C CNN
 F 1 "RC0402FR-0710RL" H 4100 4875 50  0001 C CNN
@@
 Connection ~ 3900 4650
 $Comp
-L AVR-KiCAD-Lib-Diodes:RC0402FR-0710RL R?
+L agricoltura-vine-k-rescue:RC0402FR-0710RL-AVR-KiCAD-Lib-Diodes R?
 U 1 1 5F02DC5B
 P 4100 4350
 AR Path="/5EF943A9/5F02DC5B" Ref="R?"  Part="1"
 AR Path="/5F0125AE/5F02DC5B" Ref="R22"  Part="1"
+AR Path="/5F02DC5B" Ref="R22"  Part="1"
 F 0 "R22" H 4100 4450 50  0000 C CNN
 F 1 "RC0402FR-0710RL" H 4100 4575 50  0001 C CNN
@@
 $EndComp
 $Comp
-L AVR-KiCAD-Lib-Diodes:RC0402FR-0710RL R?
+L agricoltura-vine-k-rescue:RC0402FR-0710RL-AVR-KiCAD-Lib-Diodes R?
 U 1 1 5F02DCA1
 P 4100 5950
 AR Path="/5EF943A9/5F02DCA1" Ref="R?"  Part="1"
 AR Path="/5F0125AE/5F02DCA1" Ref="R25"  Part="1"
+AR Path="/5F02DCA1" Ref="R25"  Part="1"
 F 0 "R25" H 4100 6050 50  0000 C CNN
 F 1 "RC0402FR-0710RL" H 4100 6175 50  0001 C CNN
@@
 Connection ~ 3900 5950
 $Comp
-L AVR-KiCAD-Lib-Diodes:RC0402FR-0710RL R?
+L agricoltura-vine-k-rescue:RC0402FR-0710RL-AVR-KiCAD-Lib-Diodes R?
 U 1 1 5F02DCC6
 P 4100 5650
 AR Path="/5EF943A9/5F02DCC6" Ref="R?"  Part="1"
 AR Path="/5F0125AE/5F02DCC6" Ref="R24"  Part="1"
+AR Path="/5F02DCC6" Ref="R24"  Part="1"
 F 0 "R24" H 4100 5750 50  0000 C CNN
 F 1 "RC0402FR-0710RL" H 4100 5875 50  0001 C CNN
@@
 $EndComp
 $Comp
-L AVR-KiCAD-Lib-Diodes:RC0402FR-0710RL R?
+L agricoltura-vine-k-rescue:RC0402FR-0710RL-AVR-KiCAD-Lib-Diodes R?
 U 1 1 5F0B3FED
 P 8900 4000
 AR Path="/5EF943A9/5F0B3FED" Ref="R?"  Part="1"
 AR Path="/5F0125AE/5F0B3FED" Ref="R27"  Part="1"
+AR Path="/5F0B3FED" Ref="R27"  Part="1"
 F 0 "R27" H 8900 4100 50  0000 C CNN
 F 1 "RC0402FR-0710RL" H 8900 4225 50  0001 C CNN
@@
 Connection ~ 8700 4000
 $Comp
-L AVR-KiCAD-Lib-Diodes:RC0402FR-0710RL R?
+L agricoltura-vine-k-rescue:RC0402FR-0710RL-AVR-KiCAD-Lib-Diodes R?
 U 1 1 5F0B400E
 P 8900 3700
 AR Path="/5EF943A9/5F0B400E" Ref="R?"  Part="1"
 AR Path="/5F0125AE/5F0B400E" Ref="R26"  Part="1"
+AR Path="/5F0B400E" Ref="R26"  Part="1"
 F 0 "R26" H 8900 3800 50  0000 C CNN
 F 1 "RC0402FR-0710RL" H 8900 3925 50  0001 C CNN
